Commit message: force diffusion work better

File: assert/ur_description/urdf/ur5_robot_sensor_pos2_stand_eelink.urdf (robot description, URDF)
Before this commit: robot ur5, 13 links, 12 joints
Links:
- link FT_link: geometry collision cylinder length=0.05 radius=0.008980000000; visual cylinder length=0.05 radius=0.008980000000
