Commit message: multi view camera observe encoder and position-orientation action work

File: assert/ur_description/urdf/ur5_robot_sensor_eelink_triangle.urdf (robot description, URDF)
Before this commit: robot ur5, 13 links, 12 joints
Links:
- link FT_link: geometry collision mesh filename=package://triangle/meshes/base_link.STL scale=0.9 0.9 0.9; visual mesh filename=package://triangle/meshes/base_link.STL scale=0.9 0.9 0.9

Commit message: hierarchical reforcement learning with diffusion policy on task adjust orientation and insertion work well

File: assert/ur_description/urdf/ur5_robot_sensor_eelink_triangle.urdf (robot description, URDF)
Before this commit: robot ur5, 13 links, 12 joints
Links:
- link FT_link: mass 0.15 -> 0.015; geometry collision mesh filename=package://triangle2/meshes/base_link.STL scale=0.9 0.9 0.9; visual mesh filename=package://triangle2/meshes/base_link.STL scale=0.9 0.9 0.9

Commit message: add force for collect dataset

File: assert/ur_description/urdf/ur5_robot_sensor_eelink_triangle.urdf (robot description, URDF)
Before this commit: robot ur5, 13 links, 12 joints
Links:
- link FT_link: geometry collision mesh filename=package://triangle2/meshes/base_link.STL scale=0.8 0.8 0.8; visual mesh filename=package://triangle2/meshes/base_link.STL scale=0.8 0.8 0.8
Joints:
- joint FT_joint: origin xyz=0.045 0 0 rpy=0 -1.57079632679 0 -> xyz=0.047 0 0 rpy=0 -1.57079632679 0

Commit message: hybrid position and force controller work better

File: assert/ur_description/urdf/ur5_robot_sensor_eelink_triangle.urdf (robot description, URDF)
Before this commit: robot ur5, 13 links, 12 joints
Links:
- link FT_link: geometry collision mesh filename=package://triangle2/meshes/base_link.STL scale=0.9 0.9 0.9; visual mesh filename=package://triangle2/meshes/base_link.STL scale=0.9 0.9 0.9

Commit message: plot eval result and modify urdf parameter

File: assert/ur_description/urdf/ur5_robot_sensor_eelink_triangle.urdf (robot description, URDF)
Before this commit: robot ur5, 13 links, 12 joints
Links:
- link FT_link: geometry collision mesh filename=package://triangle2/meshes/base_link.STL scale=0.97 0.97 0.97; visual mesh filename=package://triangle2/meshes/base_link.STL scale=0.97 0.97 0.97
Joints:
- joint FT_joint: origin xyz=0.047 0 0 rpy=0 -1.57079632679 0 -> xyz=0.053 0 0 rpy=0 -1.57079632679 0

Commit message: add function for plotting force/torque on insertion phase

File: assert/ur_description/urdf/ur5_robot_sensor_eelink_triangle.urdf (robot description, URDF)
Before this commit: robot ur5, 13 links, 12 joints
Links:
- link FT_link: geometry collision mesh filename=package://triangle2/meshes/base_link.STL scale=0.98 0.98 0.98; visual mesh filename=package://triangle2/meshes/base_link.STL scale=0.98 0.98 0.98

Commit message: experiment result including trajectory and force/torque for phase insertion

File: assert/ur_description/urdf/ur5_robot_sensor_eelink_triangle.urdf (robot description, URDF)
Before this commit: robot ur5, 13 links, 12 joints
Links:
- link FT_link: geometry collision mesh filename=package://triangle2/meshes/base_link.STL scale=0.99 0.99 0.99; visual mesh filename=package://triangle2/meshes/base_link.STL scale=0.99 0.99 0.99
