Commit message: plot collect dataset result for irregular peg-hole

File: assert/ur_description/urdf/ur5_robot_sensor_eelink_irregular.urdf (robot description, URDF)
Before this commit: robot ur5, 13 links, 12 joints
Links:
- link FT_link: geometry collision mesh filename=package://irregular/meshes/base_link.STL scale=0.820 0.820 0.820; visual mesh filename=package://irregular/meshes/base_link.STL scale=0.820 0.820 0.820
